File: schematics/light/light.kicad_pcb (KiCad board)
At the start: 2 copper layers, 5 parts, among them IC1 ATTINY85-P, P1 CONN_4X2

Commit message: Update light sensor schematics
Changed lines of the file:
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@@
   (general
     (links 13)
-    (no_connects 1)
-    (area 0 0 0 0)
+    (no_connects 0)
+    (area 29.845 24.765 64.135001 43.180001)
     (thickness 1.6)
     (drawings 0)
@@
   (segment (start 48.895 28.575) (end 45.72 28.575) (width 0.254) (layer B.Cu) (net 6))
   (segment (start 50.165 29.845) (end 48.895 28.575) (width 0.254) (layer B.Cu) (net 6))
-  (segment (start 50.165 35.56) (end 53.975 35.56) (width 0.254) (layer B.Cu) (net 7) (status 400000))
-  (segment (start 55.245 36.83) (end 55.245 38.1) (width 0.254) (layer B.Cu) (net 7) (status 800000))
+  (segment (start 50.165 35.56) (end 53.975 35.56) (width 0.254) (layer B.Cu) (net 7))
+  (segment (start 55.245 36.83) (end 55.245 38.1) (width 0.254) (layer B.Cu) (net 7))
   (segment (start 53.975 35.56) (end 55.245 36.83) (width 0.254) (layer B.Cu) (net 7))
-  (segment (start 55.245 38.1) (end 55.245 40.64) (width 0.254) (layer B.Cu) (net 7) (status 400000))
+  (segment (start 55.245 38.1) (end 55.245 40.64) (width 0.254) (layer B.Cu) (net 7))
   (segment (start 55.245 40.64) (end 53.34 42.545) (width 0.254) (layer B.Cu) (net 7))
   (segment (start 53.34 42.545) (end 41.91 42.545) (width 0.254) (layer B.Cu) (net 7))
   (segment (start 41.91 42.545) (end 38.735 39.37) (width 0.254) (layer B.Cu) (net 7))
-  (segment (start 38.735 39.37) (end 38.735 38.1) (width 0.254) (layer B.Cu) (net 7) (status 800000))
-  (segment (start 55.245 38.1) (end 57.785 38.1) (width 0.254) (layer B.Cu) (net 7) (status 400000))
-  (segment (start 60.325 35.56) (end 60.325 32.385) (width 0.254) (layer B.Cu) (net 7) (status 800000))
+  (segment (start 38.735 39.37) (end 38.735 38.1) (width 0.254) (layer B.Cu) (net 7))
+  (segment (start 55.245 38.1) (end 57.785 38.1) (width 0.254) (layer B.Cu) (net 7))
+  (segment (start 60.325 35.56) (end 60.325 32.385) (width 0.254) (layer B.Cu) (net 7))
   (segment (start 57.785 38.1) (end 60.325 35.56) (width 0.254) (layer B.Cu) (net 7))
   (zone (net 2) (net_name GND) (layer B.Cu) (hatch edge 0.508)
@@
     (polygon
       (pts
-        (xy 29.845 24.765) (xy 29.845 43.18) (xy 64.135 43.18) (xy 64.135 24.765)
+        (xy 29.21 45.085) (xy 63.5 45.085) (xy 63.5 24.13) (xy 29.21 24.13)
       )
     )
